Commit message: Changed urdf to include planar motion

File: urdf/block.xacro.urdf (robot description, URDF)
Before this commit: robot block, 3 links, 2 joints
Links:
- added link cuboid_y, mass 1
- link base_link: geometry collision box size=100 100 0.05; visual box size=100 100 0.05
- link cuboid: geometry collision box size=1 1 0.1; visual box size=1 1 0.1
Joints:
- added joint slider_y: type prismatic, parent base_link, child cuboid_y, origin xyz=0.0 0.0 0.1, axis 0 1 0, limit lower=-50 upper=50 effort=1000.0 velocity=300
- joint slider: limit lower=-15 upper=15 effort=1000.0 velocity=30 -> lower=-50 upper=50 effort=1000.0 velocity=300; parent base_link -> cuboid_y

File: urdf/block_acc.xacro.urdf (robot description, URDF)
Before this commit: robot block, 3 links, 2 joints
Links:
- link cuboid: geometry collision box size=1 1 0.1; visual box size=1 1 0.1
